File: lovemeter.brd (EAGLE design)
At the start: 68.6 x 53.3 mm, 9 parts

Commit message: Added code and brd
Parts:
- removed Dled: (no value), AUTODESK_CIRCUITS_BREADBOARD:LED5MM
- removed R4: 1k‎Ω, AUTODESK_CIRCUITS_BREADBOARD:0207/10
- removed Sbutton: (no value), AUTODESK_CIRCUITS_BREADBOARD:TL1105
- added D3: (no value), AUTODESK_CIRCUITS_BREADBOARD:LED5MM
- added U2: (no value), AUTODESK_CIRCUITS_BREADBOARD:TO92
- moved R1 38.1 mm to (5.00, 73.6)
- moved D2 25.4 mm to (5.00, 48.2)
- moved D1 25.4 mm to (5.00, 35.5)
- renumbered Uboard to U1
Connections:
- removed net N$10: Sbutton.2
- removed net N$11: Sbutton.1
- removed net N$5 (its old number): D2.K, R1.2
- new net N$8: D3.K, R3.2
- net N$1: now also U1.A0, U2.2; no longer R1.1, R2.1, R3.1, R4.1, U1.GND..
- net N$2: now also R1.1, R2.1, R3.1, U1.GND.., U2.1; no longer Sbutton.3, U1.5V
- net N$3: now also U1.5V, U2.3; no longer Dled.K, R4.2
- net N$4: now also D1.K, R1.2; no longer Dled.A, U1.3
- net N$6: now also D2.K, R2.2; no longer D2.A, U1.5
- net N$7: now also D2.A, U1.3; no longer D1.K, R3.2
- net N$9: now also D3.A; no longer R2.2, Sbutton.4
Changed lines of the file:
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@@
 </autorouter>
 <elements>
-<element value="" name="Uboard" library="AUTODESK_CIRCUITS_BREADBOARD" package="ARDUINO_UNO" x="5" y="10.08"></element><element value="" name="Dled" library="AUTODESK_CIRCUITS_BREADBOARD" package="LED5MM" x="5" y="22.78"></element><element value="1k‎Ω" name="R1" library="AUTODESK_CIRCUITS_BREADBOARD" package="0207/10" x="5" y="35.480000000000004"></element><element value="" name="Sbutton" library="AUTODESK_CIRCUITS_BREADBOARD" package="TL1105" x="5" y="48.18"></element><element value="" name="D1" library="AUTODESK_CIRCUITS_BREADBOARD" package="LED5MM" x="5" y="60.879999999999995"></element><element value="" name="D2" library="AUTODESK_CIRCUITS_BREADBOARD" package="LED5MM" x="5" y="73.58"></element><element value="1k‎Ω" name="R2" library="AUTODESK_CIRCUITS_BREADBOARD" package="0207/10" x="5" y="86.28"></element><element value="1k‎Ω" name="R3" library="AUTODESK_CIRCUITS_BREADBOARD" package="0207/10" x="5" y="98.98"></element><element value="1k‎Ω" name="R4" library="AUTODESK_CIRCUITS_BREADBOARD" package="0207/10" x="5" y="111.68"></element></elements>
+<element value="" name="U1" library="AUTODESK_CIRCUITS_BREADBOARD" package="ARDUINO_UNO" x="5" y="10.08"></element><element value="" name="U2" library="AUTODESK_CIRCUITS_BREADBOARD" package="TO92" x="5" y="22.78"></element><element value="" name="D1" library="AUTODESK_CIRCUITS_BREADBOARD" package="LED5MM" x="5" y="35.480000000000004"></element><element value="" name="D2" library="AUTODESK_CIRCUITS_BREADBOARD" package="LED5MM" x="5" y="48.18"></element><element value="" name="D3" library="AUTODESK_CIRCUITS_BREADBOARD" package="LED5MM" x="5" y="60.879999999999995"></element><element value="1k‎Ω" name="R1" library="AUTODESK_CIRCUITS_BREADBOARD" package="0207/10" x="5" y="73.58"></element><element value="1k‎Ω" name="R2" library="AUTODESK_CIRCUITS_BREADBOARD" package="0207/10" x="5" y="86.28"></element><element value="1k‎Ω" name="R3" library="AUTODESK_CIRCUITS_BREADBOARD" package="0207/10" x="5" y="98.98"></element></elements>
 <signals>
-<signal name="N$1"><contactref element="Uboard" pad="GND.."></contactref><contactref element="R2" pad="1"></contactref><wire x1="45.64" y1="12.620000000000001" x2="-0.08000000000000007" y2="86.28" width="0" layer="19" extent="1-1"></wire><contactref element="R1" pad="1"></contactref><wire x1="-0.08000000000000007" y1="86.28" x2="-0.08000000000000007" y2="35.480000000000004" width="0" layer="19" extent="1-1"></wire><contactref element="R3" pad="1"></contactref><wire x1="-0.08000000000000007" y1="35.480000000000004" x2="-0.08000000000000007" y2="98.98" width="0" layer="19" extent="1-1"></wire><contactref element="R4" pad="1"></contactref><wire x1="-0.08000000000000007" y1="98.98" x2="-0.08000000000000007" y2="111.68" width="0" layer="19" extent="1-1"></wire></signal><signal name="N$2"><contactref element="Uboard" pad="5V"></contactref><contactref element="Sbutton" pad="3"></contactref><wire x1="43.1" y1="12.620000000000001" x2="2.75" y2="44.93" width="0" layer="19" extent="1-1"></wire></signal><signal name="N$3"><contactref element="Dled" pad="K"></contactref><contactref element="R4" pad="2"></contactref><wire x1="6.27" y1="22.78" x2="10.08" y2="111.68" width="0" layer="19" extent="1-1"></wire></signal><signal name="N$4"><contactref element="Dled" pad="A"></contactref><contactref element="Uboard" pad="3"></contactref><wire x1="3.73" y1="22.78" x2="60.88" y2="60.879999999999995" width="0" layer="19" extent="1-1"></wire></signal><signal name="N$5"><contactref element="D2" pad="K"></contactref><contactref element="R1" pad="2"></contactref><wire x1="6.27" y1="73.58" x2="10.08" y2="35.480000000000004" width="0" layer="19" extent="1-1"></wire></signal><signal name="N$6"><contactref element="D2" pad="A"></contactref><contactref element="Uboard" pad="5"></contactref><wire x1="3.73" y1="73.58" x2="55.8" y2="60.879999999999995" width="0" layer="19" extent="1-1"></wire></signal><signal name="N$7"><contactref element="D1" pad="K"></contactref><contactref element="R3" pad="2"></contactref><wire x1="6.27" y1="60.879999999999995" x2="10.08" y2="98.98" width="0" layer="19" extent="1-1"></wire></signal><signal name="N$8"><contactref element="D1" pad="A"></contactref><contactref element="Uboard" pad="4"></contactref><wire x1="3.73" y1="60.879999999999995" x2="58.34" y2="60.879999999999995" width="0" layer="19" extent="1-1"></wire></signal><signal name="N$9"><contactref element="Sbutton" pad="4"></contactref><contactref element="Uboard" pad="2"></contactref><wire x1="7.25" y1="44.93" x2="63.42" y2="60.879999999999995" width="0" layer="19" extent="1-1"></wire><contactref element="R2" pad="2"></contactref><wire x1="63.42" y1="60.879999999999995" x2="10.08" y2="86.28" width="0" layer="19" extent="1-1"></wire></signal><signal name="N$10"><contactref element="Sbutton" pad="2"></contactref></signal><signal name="N$11"><contactref element="Sbutton" pad="1"></contactref></signal></signals>
+<signal name="N$1"><contactref element="U2" pad="2"></contactref><contactref element="U1" pad="A0"></contactref><wire x1="5" y1="24.685000000000002" x2="55.8" y2="12.620000000000001" width="0" layer="19" extent="1-1"></wire></signal><signal name="N$2"><contactref element="U2" pad="1"></contactref><contactref element="U1" pad="GND.."></contactref><wire x1="6.27" y1="22.78" x2="45.64" y2="12.620000000000001" width="0" layer="19" extent="1-1"></wire><contactref element="R1" pad="1"></contactref><wire x1="45.64" y1="12.620000000000001" x2="-0.08000000000000007" y2="73.58" width="0" layer="19" extent="1-1"></wire><contactref element="R2" pad="1"></contactref><wire x1="-0.08000000000000007" y1="73.58" x2="-0.08000000000000007" y2="86.28" width="0" layer="19" extent="1-1"></wire><contactref element="R3" pad="1"></contactref><wire x1="-0.08000000000000007" y1="86.28" x2="-0.08000000000000007" y2="98.98" width="0" layer="19" extent="1-1"></wire></signal><signal name="N$3"><contactref element="U2" pad="3"></contactref><contactref element="U1" pad="5V"></contactref><wire x1="3.73" y1="22.78" x2="43.1" y2="12.620000000000001" width="0" layer="19" extent="1-1"></wire></signal><signal name="N$4"><contactref element="D1" pad="K"></contactref><contactref element="R1" pad="2"></contactref><wire x1="6.27" y1="35.480000000000004" x2="10.08" y2="73.58" width="0" layer="19" extent="1-1"></wire></signal><signal name="N$5"><contactref element="D1" pad="A"></contactref><contactref element="U1" pad="4"></contactref><wire x1="3.73" y1="35.480000000000004" x2="58.34" y2="60.879999999999995" width="0" layer="19" extent="1-1"></wire></signal><signal name="N$6"><contactref element="D2" pad="K"></contactref><contactref element="R2" pad="2"></contactref><wire x1="6.27" y1="48.18" x2="10.08" y2="86.28" width="0" layer="19" extent="1-1"></wire></signal><signal name="N$7"><contactref element="D2" pad="A"></contactref><contactref element="U1" pad="3"></contactref><wire x1="3.73" y1="48.18" x2="60.88" y2="60.879999999999995" width="0" layer="19" extent="1-1"></wire></signal><signal name="N$8"><contactref element="D3" pad="K"></contactref><contactref element="R3" pad="2"></contactref><wire x1="6.27" y1="60.879999999999995" x2="10.08" y2="98.98" width="0" layer="19" extent="1-1"></wire></signal><signal name="N$9"><contactref element="D3" pad="A"></contactref><contactref element="U1" pad="2"></contactref><wire x1="3.73" y1="60.879999999999995" x2="63.42" y2="60.879999999999995" width="0" layer="19" extent="1-1"></wire></signal></signals>
 </board>
 </drawing>
