File: color-mixing-lamp.brd (EAGLE design)
At the start: 68.6 x 53.3 mm, 9 parts

Commit message: Added code and brd
Parts:
- removed D2, Dled: (no value), AUTODESK_CIRCUITS_BREADBOARD:LED5MM
- removed Sbutton: (no value), AUTODESK_CIRCUITS_BREADBOARD:TL1105
- added R5, R6: (no value), AUTODESK_CIRCUITS_BREADBOARD:PHOTORESISTOR-2.54
- added R7, R8, R9: 10000‎Ω, AUTODESK_CIRCUITS_BREADBOARD:0207/10
- D1: device AUTODESK_CIRCUITS_BREADBOARD:LED5MM -> AUTODESK_CIRCUITS_BREADBOARD:LED-RGB-THRU
- R4: value 1k‎Ω -> (none); device AUTODESK_CIRCUITS_BREADBOARD:0207/10 -> AUTODESK_CIRCUITS_BREADBOARD:PHOTORESISTOR-2.54
- moved R3 38.1 mm to (5.00, 60.9)
- moved R4 38.1 mm to (5.00, 73.6)
- moved R2 38.1 mm to (5.00, 48.2)
- moved D1 38.1 mm to (5.00, 22.8)
- renumbered Uboard to U1
Connections:
- net N$1: now also D1.2, R7.2, R8.2, R9.2; no longer R1.1, R2.1, R3.1, R4.1
- net N$10: now also R6.P$1, R9.1, U1.A0; no longer Sbutton.2
- net N$11: now also R4.P$2, R5.P$2, R6.P$2, U1.5V; no longer Sbutton.1
- net N$2: now also D1.3, R2.2; no longer Sbutton.3, U1.5V
- net N$3: now also D1.4, R3.2; no longer Dled.K, R4.2
- net N$4: now also D1.1, R1.2; no longer Dled.A, U1.3
- net N$5: now also R1.1, U1.10; no longer D2.K, R1.2
- net N$6: now also R2.1, U1.11; no longer D2.A, U1.5
- net N$7: now also R3.1, U1.9; no longer D1.K, R3.2
- net N$8: now also R4.P$1, R7.1, U1.A2; no longer D1.A, U1.4
- net N$9: now also R5.P$1, R8.1, U1.A1; no longer R2.2, Sbutton.4, U1.2
Changed lines of the file:
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@@
 </autorouter>
 <elements>
-<element value="" name="Uboard" library="AUTODESK_CIRCUITS_BREADBOARD" package="ARDUINO_UNO" x="5" y="10.08"></element><element value="" name="Dled" library="AUTODESK_CIRCUITS_BREADBOARD" package="LED5MM" x="5" y="22.78"></element><element value="1k‎Ω" name="R1" library="AUTODESK_CIRCUITS_BREADBOARD" package="0207/10" x="5" y="35.480000000000004"></element><element value="" name="Sbutton" library="AUTODESK_CIRCUITS_BREADBOARD" package="TL1105" x="5" y="48.18"></element><element value="" name="D1" library="AUTODESK_CIRCUITS_BREADBOARD" package="LED5MM" x="5" y="60.879999999999995"></element><element value="" name="D2" library="AUTODESK_CIRCUITS_BREADBOARD" package="LED5MM" x="5" y="73.58"></element><element value="1k‎Ω" name="R2" library="AUTODESK_CIRCUITS_BREADBOARD" package="0207/10" x="5" y="86.28"></element><element value="1k‎Ω" name="R3" library="AUTODESK_CIRCUITS_BREADBOARD" package="0207/10" x="5" y="98.98"></element><element value="1k‎Ω" name="R4" library="AUTODESK_CIRCUITS_BREADBOARD" package="0207/10" x="5" y="111.68"></element></elements>
+<element value="" name="U1" library="AUTODESK_CIRCUITS_BREADBOARD" package="ARDUINO_UNO" x="5" y="10.08"></element><element value="" name="D1" library="AUTODESK_CIRCUITS_BREADBOARD" package="LED-RGB-THRU" x="5" y="22.78"></element><element value="1k‎Ω" name="R1" library="AUTODESK_CIRCUITS_BREADBOARD" package="0207/10" x="5" y="35.480000000000004"></element><element value="1k‎Ω" name="R2" library="AUTODESK_CIRCUITS_BREADBOARD" package="0207/10" x="5" y="48.18"></element><element value="1k‎Ω" name="R3" library="AUTODESK_CIRCUITS_BREADBOARD" package="0207/10" x="5" y="60.879999999999995"></element><element value="" name="R4" library="AUTODESK_CIRCUITS_BREADBOARD" package="PHOTORESISTOR-2.54" x="5" y="73.58"></element><element value="" name="R5" library="AUTODESK_CIRCUITS_BREADBOARD" package="PHOTORESISTOR-2.54" x="5" y="86.28"></element><element value="" name="R6" library="AUTODESK_CIRCUITS_BREADBOARD" package="PHOTORESISTOR-2.54" x="5" y="98.98"></element><element value="10000‎Ω" name="R7" library="AUTODESK_CIRCUITS_BREADBOARD" package="0207/10" x="5" y="111.68"></element><element value="10000‎Ω" name="R8" library="AUTODESK_CIRCUITS_BREADBOARD" package="0207/10" x="5" y="124.38000000000001"></element><element value="10000‎Ω" name="R9" library="AUTODESK_CIRCUITS_BREADBOARD" package="0207/10" x="5" y="137.08"></element></elements>
 <signals>
-<signal name="N$1"><contactref element="Uboard" pad="GND.."></contactref><contactref element="R2" pad="1"></contactref><wire x1="45.64" y1="12.620000000000001" x2="-0.08000000000000007" y2="86.28" width="0" layer="19" extent="1-1"></wire><contactref element="R1" pad="1"></contactref><wire x1="-0.08000000000000007" y1="86.28" x2="-0.08000000000000007" y2="35.480000000000004" width="0" layer="19" extent="1-1"></wire><contactref element="R3" pad="1"></contactref><wire x1="-0.08000000000000007" y1="35.480000000000004" x2="-0.08000000000000007" y2="98.98" width="0" layer="19" extent="1-1"></wire><contactref element="R4" pad="1"></contactref><wire x1="-0.08000000000000007" y1="98.98" x2="-0.08000000000000007" y2="111.68" width="0" layer="19" extent="1-1"></wire></signal><signal name="N$2"><contactref element="Uboard" pad="5V"></contactref><contactref element="Sbutton" pad="3"></contactref><wire x1="43.1" y1="12.620000000000001" x2="2.75" y2="44.93" width="0" layer="19" extent="1-1"></wire></signal><signal name="N$3"><contactref element="Dled" pad="K"></contactref><contactref element="R4" pad="2"></contactref><wire x1="6.27" y1="22.78" x2="10.08" y2="111.68" width="0" layer="19" extent="1-1"></wire></signal><signal name="N$4"><contactref element="Dled" pad="A"></contactref><contactref element="Uboard" pad="3"></contactref><wire x1="3.73" y1="22.78" x2="60.88" y2="60.879999999999995" width="0" layer="19" extent="1-1"></wire></signal><signal name="N$5"><contactref element="D2" pad="K"></contactref><contactref element="R1" pad="2"></contactref><wire x1="6.27" y1="73.58" x2="10.08" y2="35.480000000000004" width="0" layer="19" extent="1-1"></wire></signal><signal name="N$6"><contactref element="D2" pad="A"></contactref><contactref element="Uboard" pad="5"></contactref><wire x1="3.73" y1="73.58" x2="55.8" y2="60.879999999999995" width="0" layer="19" extent="1-1"></wire></signal><signal name="N$7"><contactref element="D1" pad="K"></contactref><contactref element="R3" pad="2"></contactref><wire x1="6.27" y1="60.879999999999995" x2="10.08" y2="98.98" width="0" layer="19" extent="1-1"></wire></signal><signal name="N$8"><contactref element="D1" pad="A"></contactref><contactref element="Uboard" pad="4"></contactref><wire x1="3.73" y1="60.879999999999995" x2="58.34" y2="60.879999999999995" width="0" layer="19" extent="1-1"></wire></signal><signal name="N$9"><contactref element="Sbutton" pad="4"></contactref><contactref element="Uboard" pad="2"></contactref><wire x1="7.25" y1="44.93" x2="63.42" y2="60.879999999999995" width="0" layer="19" extent="1-1"></wire><contactref element="R2" pad="2"></contactref><wire x1="63.42" y1="60.879999999999995" x2="10.08" y2="86.28" width="0" layer="19" extent="1-1"></wire></signal><signal name="N$10"><contactref element="Sbutton" pad="2"></contactref></signal><signal name="N$11"><contactref element="Sbutton" pad="1"></contactref></signal></signals>
+<signal name="N$1"><contactref element="U1" pad="GND.."></contactref><contactref element="D1" pad="2"></contactref><wire x1="45.64" y1="12.620000000000001" x2="5.635" y2="22.78" width="0" layer="19" extent="1-1"></wire><contactref element="R9" pad="2"></contactref><wire x1="5.635" y1="22.78" x2="10.08" y2="137.08" width="0" layer="19" extent="1-1"></wire><contactref element="R8" pad="2"></contactref><wire x1="10.08" y1="137.08" x2="10.08" y2="124.38000000000001" width="0" layer="19" extent="1-1"></wire><contactref element="R7" pad="2"></contactref><wire x1="10.08" y1="124.38000000000001" x2="10.08" y2="111.68" width="0" layer="19" extent="1-1"></wire></signal><signal name="N$2"><contactref element="D1" pad="3"></contactref><contactref element="R2" pad="2"></contactref><wire x1="4.365" y1="22.78" x2="10.08" y2="48.18" width="0" layer="19" extent="1-1"></wire></signal><signal name="N$3"><contactref element="D1" pad="4"></contactref><contactref element="R3" pad="2"></contactref><wire x1="3.0949999999999998" y1="22.78" x2="10.08" y2="60.879999999999995" width="0" layer="19" extent="1-1"></wire></signal><signal name="N$4"><contactref element="D1" pad="1"></contactref><contactref element="R1" pad="2"></contactref><wire x1="6.905" y1="22.78" x2="10.08" y2="35.480000000000004" width="0" layer="19" extent="1-1"></wire></signal><signal name="N$5"><contactref element="R1" pad="1"></contactref><contactref element="U1" pad="10"></contactref><wire x1="-0.08000000000000007" y1="35.480000000000004" x2="41.576" y2="60.879999999999995" width="0" layer="19" extent="1-1"></wire></signal><signal name="N$6"><contactref element="R2" pad="1"></contactref><contactref element="U1" pad="11"></contactref><wire x1="-0.08000000000000007" y1="48.18" x2="39.036" y2="60.879999999999995" width="0" layer="19" extent="1-1"></wire></signal><signal name="N$7"><contactref element="R3" pad="1"></contactref><contactref element="U1" pad="9"></contactref><wire x1="-0.08000000000000007" y1="60.879999999999995" x2="44.116" y2="60.879999999999995" width="0" layer="19" extent="1-1"></wire></signal><signal name="N$8"><contactref element="R4" pad="P$1"></contactref><contactref element="R7" pad="1"></contactref><wire x1="3.73" y1="73.58" x2="-0.08000000000000007" y2="111.68" width="0" layer="19" extent="1-1"></wire><contactref element="U1" pad="A2"></contactref><wire x1="-0.08000000000000007" y1="111.68" x2="60.88" y2="12.620000000000001" width="0" layer="19" extent="1-1"></wire></signal><signal name="N$9"><contactref element="R5" pad="P$1"></contactref><contactref element="R8" pad="1"></contactref><wire x1="3.73" y1="86.28" x2="-0.08000000000000007" y2="124.38000000000001" width="0" layer="19" extent="1-1"></wire><contactref element="U1" pad="A1"></contactref><wire x1="-0.08000000000000007" y1="124.38000000000001" x2="58.34" y2="12.620000000000001" width="0" layer="19" extent="1-1"></wire></signal><signal name="N$10"><contactref element="R6" pad="P$1"></contactref><contactref element="R9" pad="1"></contactref><wire x1="3.73" y1="98.98" x2="-0.08000000000000007" y2="137.08" width="0" layer="19" extent="1-1"></wire><contactref element="U1" pad="A0"></contactref><wire x1="-0.08000000000000007" y1="137.08" x2="55.8" y2="12.620000000000001" width="0" layer="19" extent="1-1"></wire></signal><signal name="N$11"><contactref element="R6" pad="P$2"></contactref><contactref element="R5" pad="P$2"></contactref><wire x1="6.27" y1="98.98" x2="6.27" y2="86.28" width="0" layer="19" extent="1-1"></wire><contactref element="R4" pad="P$2"></contactref><wire x1="6.27" y1="86.28" x2="6.27" y2="73.58" width="0" layer="19" extent="1-1"></wire><contactref element="U1" pad="5V"></contactref><wire x1="6.27" y1="73.58" x2="43.1" y2="12.620000000000001" width="0" layer="19" extent="1-1"></wire></signal></signals>
 </board>
 </drawing>
