File: light-theremin.brd (EAGLE design)
At the start: 68.6 x 53.3 mm, 9 parts

Commit message: Added code and brd
Parts:
- removed D1, D2, Dled: (no value), AUTODESK_CIRCUITS_BREADBOARD:LED5MM
- removed R3, R4: 1k‎Ω, AUTODESK_CIRCUITS_BREADBOARD:0207/10
- removed Sbutton: (no value), AUTODESK_CIRCUITS_BREADBOARD:TL1105
- added PIEZO1: (no value), AUTODESK_CIRCUITS_BREADBOARD:PIEZO-22MM
- R1: value 1k‎Ω -> (none); device AUTODESK_CIRCUITS_BREADBOARD:0207/10 -> AUTODESK_CIRCUITS_BREADBOARD:PHOTORESISTOR-2.54
- R2: value 1k‎Ω -> 10000‎Ω
- moved R2 38.1 mm to (5.00, 48.2)
- renumbered Uboard to U1
Connections:
- removed net N$10: Sbutton.2
- removed net N$11: Sbutton.1
- removed net N$5: D2.K, R1.2
- removed net N$6: D2.A, U1.5
- removed net N$7: D1.K, R3.2
- removed net N$8: D1.A, U1.4
- removed net N$9: R2.2, Sbutton.4, U1.2
- net N$1: now also PIEZO1.P$1, R2.2; no longer R1.1, R2.1, R3.1, R4.1
- net N$2: now also PIEZO1.P$2, U1.8; no longer Sbutton.3, U1.5V
- net N$3: now also R1.P$2, R2.1, U1.A0; no longer Dled.K, R4.2
- net N$4: now also R1.P$1, U1.5V; no longer Dled.A, U1.3
Changed lines of the file:
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@@
 </autorouter>
 <elements>
-<element value="" name="Uboard" library="AUTODESK_CIRCUITS_BREADBOARD" package="ARDUINO_UNO" x="5" y="10.08"></element><element value="" name="Dled" library="AUTODESK_CIRCUITS_BREADBOARD" package="LED5MM" x="5" y="22.78"></element><element value="1k‎Ω" name="R1" library="AUTODESK_CIRCUITS_BREADBOARD" package="0207/10" x="5" y="35.480000000000004"></element><element value="" name="Sbutton" library="AUTODESK_CIRCUITS_BREADBOARD" package="TL1105" x="5" y="48.18"></element><element value="" name="D1" library="AUTODESK_CIRCUITS_BREADBOARD" package="LED5MM" x="5" y="60.879999999999995"></element><element value="" name="D2" library="AUTODESK_CIRCUITS_BREADBOARD" package="LED5MM" x="5" y="73.58"></element><element value="1k‎Ω" name="R2" library="AUTODESK_CIRCUITS_BREADBOARD" package="0207/10" x="5" y="86.28"></element><element value="1k‎Ω" name="R3" library="AUTODESK_CIRCUITS_BREADBOARD" package="0207/10" x="5" y="98.98"></element><element value="1k‎Ω" name="R4" library="AUTODESK_CIRCUITS_BREADBOARD" package="0207/10" x="5" y="111.68"></element></elements>
+<element value="" name="U1" library="AUTODESK_CIRCUITS_BREADBOARD" package="ARDUINO_UNO" x="5" y="10.08"></element><element value="" name="PIEZO1" library="AUTODESK_CIRCUITS_BREADBOARD" package="PIEZO-22MM" x="5" y="22.78"></element><element value="" name="R1" library="AUTODESK_CIRCUITS_BREADBOARD" package="PHOTORESISTOR-2.54" x="5" y="35.480000000000004"></element><element value="10000‎Ω" name="R2" library="AUTODESK_CIRCUITS_BREADBOARD" package="0207/10" x="5" y="48.18"></element></elements>
 <signals>
-<signal name="N$1"><contactref element="Uboard" pad="GND.."></contactref><contactref element="R2" pad="1"></contactref><wire x1="45.64" y1="12.620000000000001" x2="-0.08000000000000007" y2="86.28" width="0" layer="19" extent="1-1"></wire><contactref element="R1" pad="1"></contactref><wire x1="-0.08000000000000007" y1="86.28" x2="-0.08000000000000007" y2="35.480000000000004" width="0" layer="19" extent="1-1"></wire><contactref element="R3" pad="1"></contactref><wire x1="-0.08000000000000007" y1="35.480000000000004" x2="-0.08000000000000007" y2="98.98" width="0" layer="19" extent="1-1"></wire><contactref element="R4" pad="1"></contactref><wire x1="-0.08000000000000007" y1="98.98" x2="-0.08000000000000007" y2="111.68" width="0" layer="19" extent="1-1"></wire></signal><signal name="N$2"><contactref element="Uboard" pad="5V"></contactref><contactref element="Sbutton" pad="3"></contactref><wire x1="43.1" y1="12.620000000000001" x2="2.75" y2="44.93" width="0" layer="19" extent="1-1"></wire></signal><signal name="N$3"><contactref element="Dled" pad="K"></contactref><contactref element="R4" pad="2"></contactref><wire x1="6.27" y1="22.78" x2="10.08" y2="111.68" width="0" layer="19" extent="1-1"></wire></signal><signal name="N$4"><contactref element="Dled" pad="A"></contactref><contactref element="Uboard" pad="3"></contactref><wire x1="3.73" y1="22.78" x2="60.88" y2="60.879999999999995" width="0" layer="19" extent="1-1"></wire></signal><signal name="N$5"><contactref element="D2" pad="K"></contactref><contactref element="R1" pad="2"></contactref><wire x1="6.27" y1="73.58" x2="10.08" y2="35.480000000000004" width="0" layer="19" extent="1-1"></wire></signal><signal name="N$6"><contactref element="D2" pad="A"></contactref><contactref element="Uboard" pad="5"></contactref><wire x1="3.73" y1="73.58" x2="55.8" y2="60.879999999999995" width="0" layer="19" extent="1-1"></wire></signal><signal name="N$7"><contactref element="D1" pad="K"></contactref><contactref element="R3" pad="2"></contactref><wire x1="6.27" y1="60.879999999999995" x2="10.08" y2="98.98" width="0" layer="19" extent="1-1"></wire></signal><signal name="N$8"><contactref element="D1" pad="A"></contactref><contactref element="Uboard" pad="4"></contactref><wire x1="3.73" y1="60.879999999999995" x2="58.34" y2="60.879999999999995" width="0" layer="19" extent="1-1"></wire></signal><signal name="N$9"><contactref element="Sbutton" pad="4"></contactref><contactref element="Uboard" pad="2"></contactref><wire x1="7.25" y1="44.93" x2="63.42" y2="60.879999999999995" width="0" layer="19" extent="1-1"></wire><contactref element="R2" pad="2"></contactref><wire x1="63.42" y1="60.879999999999995" x2="10.08" y2="86.28" width="0" layer="19" extent="1-1"></wire></signal><signal name="N$10"><contactref element="Sbutton" pad="2"></contactref></signal><signal name="N$11"><contactref element="Sbutton" pad="1"></contactref></signal></signals>
+<signal name="N$1"><contactref element="U1" pad="GND.."></contactref><contactref element="PIEZO1" pad="P$1"></contactref><wire x1="45.64" y1="12.620000000000001" x2="0" y2="22.78" width="0" layer="19" extent="1-1"></wire><contactref element="R2" pad="2"></contactref><wire x1="0" y1="22.78" x2="10.08" y2="48.18" width="0" layer="19" extent="1-1"></wire></signal><signal name="N$2"><contactref element="PIEZO1" pad="P$2"></contactref><contactref element="U1" pad="8"></contactref><wire x1="10" y1="22.78" x2="46.656" y2="60.879999999999995" width="0" layer="19" extent="1-1"></wire></signal><signal name="N$3"><contactref element="R1" pad="P$2"></contactref><contactref element="R2" pad="1"></contactref><wire x1="6.27" y1="35.480000000000004" x2="-0.08000000000000007" y2="48.18" width="0" layer="19" extent="1-1"></wire><contactref element="U1" pad="A0"></contactref><wire x1="-0.08000000000000007" y1="48.18" x2="55.8" y2="12.620000000000001" width="0" layer="19" extent="1-1"></wire></signal><signal name="N$4"><contactref element="R1" pad="P$1"></contactref><contactref element="U1" pad="5V"></contactref><wire x1="3.73" y1="35.480000000000004" x2="43.1" y2="12.620000000000001" width="0" layer="19" extent="1-1"></wire></signal></signals>
 </board>
 </drawing>
