File: digital-hourglass.brd (EAGLE design)
At the start: 68.6 x 53.3 mm, 9 parts

Commit message: Added code and brd
Parts:
- removed Dled: (no value), AUTODESK_CIRCUITS_BREADBOARD:LED5MM
- removed Sbutton: (no value), AUTODESK_CIRCUITS_BREADBOARD:TL1105
- added D3, D4, D5, D6: (no value), AUTODESK_CIRCUITS_BREADBOARD:LED5MM
- added R5, R6, R7: 220‎Ω, AUTODESK_CIRCUITS_BREADBOARD:0207/10
- added TILT1: (no value), AUTODESK_CIRCUITS_BREADBOARD:SW2-12.7-12.0X3.6X3.6MM
- R1: value 1k‎Ω -> 10000‎Ω
- R2, R3, R4: value 1k‎Ω -> 220‎Ω
- moved R4 38.1 mm to (5.00, 149.8)
- moved R2 38.1 mm to (5.00, 124.4)
- moved R3 38.1 mm to (5.00, 137.1)
- moved D2 12.7 mm to (5.00, 60.9)
- moved R1 12.7 mm to (5.00, 22.8)
- moved D1 12.7 mm to (5.00, 48.2)
- renumbered Uboard to U1
Connections:
- new net N$12: D3.K, R4.1
- new net N$13: D4.K, R5.1
- new net N$14: D5.K, R6.1
- new net N$15: D6.K, R7.1
- net N$1: now also TILT1.1, U1.5V; no longer R1.1, R2.1, R3.1, R4.1, U1.GND..
- net N$10: now also D1.K, R2.1; no longer Sbutton.2
- net N$11: now also D2.K, R3.1; no longer Sbutton.1
- net N$2: now also R1.2, R2.2, R3.2, R4.2, R5.2, R6.2, R7.2, U1.GND..; no longer Sbutton.3, U1.5V
- net N$3: now also R1.1, TILT1.2, U1.8; no longer Dled.K, R4.2
- net N$4: now also D1.A, U1.7; no longer Dled.A, U1.3
- net N$5: now also D2.A, U1.6; no longer D2.K, R1.2
- net N$6: now also D3.A; no longer D2.A
- net N$7: now also D4.A, U1.4; no longer D1.K, R3.2
- net N$8: now also D5.A, U1.3; no longer D1.A, U1.4
- net N$9: now also D6.A; no longer R2.2, Sbutton.4
