File: motorized-pinwheel.brd (EAGLE design)
At the start: 68.6 x 53.3 mm, 9 parts

Commit message: Added code and brd
Parts:
- removed D2, Dled: (no value), AUTODESK_CIRCUITS_BREADBOARD:LED5MM
- removed R2, R3, R4: 1k‎Ω, AUTODESK_CIRCUITS_BREADBOARD:0207/10
- removed Sbutton: (no value), AUTODESK_CIRCUITS_BREADBOARD:TL1105
- added BAT1: (no value), AUTODESK_CIRCUITS_BREADBOARD:DC-POWER
- added S1: (no value), AUTODESK_CIRCUITS_BREADBOARD:TL1105
- added T1: (no value), AUTODESK_CIRCUITS_BREADBOARD:TO92
- D1: device AUTODESK_CIRCUITS_BREADBOARD:LED5MM -> AUTODESK_CIRCUITS_BREADBOARD:D-7.5
- R1: value 1k‎Ω -> 10000‎Ω
- moved D1 12.7 mm to (5.00, 73.6)
- moved R1 12.7 mm to (5.00, 48.2)
- renumbered Uboard to U1
Connections:
- removed net N$10: Sbutton.2
- removed net N$11: Sbutton.1
- removed net N$9: R2.2, Sbutton.4, U1.2
- net N$1: now also S1.3, U1.5V; no longer R1.1, R2.1, R3.1, R4.1, U1.GND..
- net N$2: now also R1.1, S1.4, U1.2; no longer Sbutton.3, U1.5V
- net N$3: now also S1.2; no longer Dled.K, R4.2
- net N$4: now also S1.1; no longer Dled.A, U1.3
- net N$5: now also BAT1.+, D1.A; no longer D2.K, R1.2
- net N$6: now also T1.3, U1.9; no longer D2.A, U1.5
- net N$7: now also D1.C, T1.2; no longer D1.K, R3.2
- net N$8: now also BAT1.-, R1.2, T1.1, U1.GND..; no longer D1.A, U1.4
Changed lines of the file:
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@@
 </autorouter>
 <elements>
-<element value="" name="Uboard" library="AUTODESK_CIRCUITS_BREADBOARD" package="ARDUINO_UNO" x="5" y="10.08"></element><element value="" name="Dled" library="AUTODESK_CIRCUITS_BREADBOARD" package="LED5MM" x="5" y="22.78"></element><element value="1k‎Ω" name="R1" library="AUTODESK_CIRCUITS_BREADBOARD" package="0207/10" x="5" y="35.480000000000004"></element><element value="" name="Sbutton" library="AUTODESK_CIRCUITS_BREADBOARD" package="TL1105" x="5" y="48.18"></element><element value="" name="D1" library="AUTODESK_CIRCUITS_BREADBOARD" package="LED5MM" x="5" y="60.879999999999995"></element><element value="" name="D2" library="AUTODESK_CIRCUITS_BREADBOARD" package="LED5MM" x="5" y="73.58"></element><element value="1k‎Ω" name="R2" library="AUTODESK_CIRCUITS_BREADBOARD" package="0207/10" x="5" y="86.28"></element><element value="1k‎Ω" name="R3" library="AUTODESK_CIRCUITS_BREADBOARD" package="0207/10" x="5" y="98.98"></element><element value="1k‎Ω" name="R4" library="AUTODESK_CIRCUITS_BREADBOARD" package="0207/10" x="5" y="111.68"></element></elements>
+<element value="" name="U1" library="AUTODESK_CIRCUITS_BREADBOARD" package="ARDUINO_UNO" x="5" y="10.08"></element><element value="" name="S1" library="AUTODESK_CIRCUITS_BREADBOARD" package="TL1105" x="5" y="22.78"></element><element value="" name="BAT1" library="AUTODESK_CIRCUITS_BREADBOARD" package="DC-POWER" x="5" y="35.480000000000004"></element><element value="10000‎Ω" name="R1" library="AUTODESK_CIRCUITS_BREADBOARD" package="0207/10" x="5" y="48.18"></element><element value="" name="T1" library="AUTODESK_CIRCUITS_BREADBOARD" package="TO92" x="5" y="60.879999999999995"></element><element value="" name="D1" library="AUTODESK_CIRCUITS_BREADBOARD" package="D-7.5" x="5" y="73.58"></element></elements>
 <signals>
-<signal name="N$1"><contactref element="Uboard" pad="GND.."></contactref><contactref element="R2" pad="1"></contactref><wire x1="45.64" y1="12.620000000000001" x2="-0.08000000000000007" y2="86.28" width="0" layer="19" extent="1-1"></wire><contactref element="R1" pad="1"></contactref><wire x1="-0.08000000000000007" y1="86.28" x2="-0.08000000000000007" y2="35.480000000000004" width="0" layer="19" extent="1-1"></wire><contactref element="R3" pad="1"></contactref><wire x1="-0.08000000000000007" y1="35.480000000000004" x2="-0.08000000000000007" y2="98.98" width="0" layer="19" extent="1-1"></wire><contactref element="R4" pad="1"></contactref><wire x1="-0.08000000000000007" y1="98.98" x2="-0.08000000000000007" y2="111.68" width="0" layer="19" extent="1-1"></wire></signal><signal name="N$2"><contactref element="Uboard" pad="5V"></contactref><contactref element="Sbutton" pad="3"></contactref><wire x1="43.1" y1="12.620000000000001" x2="2.75" y2="44.93" width="0" layer="19" extent="1-1"></wire></signal><signal name="N$3"><contactref element="Dled" pad="K"></contactref><contactref element="R4" pad="2"></contactref><wire x1="6.27" y1="22.78" x2="10.08" y2="111.68" width="0" layer="19" extent="1-1"></wire></signal><signal name="N$4"><contactref element="Dled" pad="A"></contactref><contactref element="Uboard" pad="3"></contactref><wire x1="3.73" y1="22.78" x2="60.88" y2="60.879999999999995" width="0" layer="19" extent="1-1"></wire></signal><signal name="N$5"><contactref element="D2" pad="K"></contactref><contactref element="R1" pad="2"></contactref><wire x1="6.27" y1="73.58" x2="10.08" y2="35.480000000000004" width="0" layer="19" extent="1-1"></wire></signal><signal name="N$6"><contactref element="D2" pad="A"></contactref><contactref element="Uboard" pad="5"></contactref><wire x1="3.73" y1="73.58" x2="55.8" y2="60.879999999999995" width="0" layer="19" extent="1-1"></wire></signal><signal name="N$7"><contactref element="D1" pad="K"></contactref><contactref element="R3" pad="2"></contactref><wire x1="6.27" y1="60.879999999999995" x2="10.08" y2="98.98" width="0" layer="19" extent="1-1"></wire></signal><signal name="N$8"><contactref element="D1" pad="A"></contactref><contactref element="Uboard" pad="4"></contactref><wire x1="3.73" y1="60.879999999999995" x2="58.34" y2="60.879999999999995" width="0" layer="19" extent="1-1"></wire></signal><signal name="N$9"><contactref element="Sbutton" pad="4"></contactref><contactref element="Uboard" pad="2"></contactref><wire x1="7.25" y1="44.93" x2="63.42" y2="60.879999999999995" width="0" layer="19" extent="1-1"></wire><contactref element="R2" pad="2"></contactref><wire x1="63.42" y1="60.879999999999995" x2="10.08" y2="86.28" width="0" layer="19" extent="1-1"></wire></signal><signal name="N$10"><contactref element="Sbutton" pad="2"></contactref></signal><signal name="N$11"><contactref element="Sbutton" pad="1"></contactref></signal></signals>
+<signal name="N$1"><contactref element="U1" pad="5V"></contactref><contactref element="S1" pad="3"></contactref><wire x1="43.1" y1="12.620000000000001" x2="2.75" y2="19.53" width="0" layer="19" extent="1-1"></wire></signal><signal name="N$2"><contactref element="S1" pad="4"></contactref><contactref element="U1" pad="2"></contactref><wire x1="7.25" y1="19.53" x2="63.42" y2="60.879999999999995" width="0" layer="19" extent="1-1"></wire><contactref element="R1" pad="1"></contactref><wire x1="63.42" y1="60.879999999999995" x2="-0.08000000000000007" y2="48.18" width="0" layer="19" extent="1-1"></wire></signal><signal name="N$3"><contactref element="S1" pad="2"></contactref></signal><signal name="N$4"><contactref element="S1" pad="1"></contactref></signal><signal name="N$5"><contactref element="BAT1" pad="+"></contactref><contactref element="D1" pad="A"></contactref><wire x1="5" y1="38.02" x2="8.81" y2="73.58" width="0" layer="19" extent="1-1"></wire></signal><signal name="N$6"><contactref element="T1" pad="3"></contactref><contactref element="U1" pad="9"></contactref><wire x1="3.73" y1="60.879999999999995" x2="44.116" y2="60.879999999999995" width="0" layer="19" extent="1-1"></wire></signal><signal name="N$7"><contactref element="T1" pad="2"></contactref><contactref element="D1" pad="C"></contactref><wire x1="5" y1="62.785" x2="1.19" y2="73.58" width="0" layer="19" extent="1-1"></wire></signal><signal name="N$8"><contactref element="T1" pad="1"></contactref><contactref element="R1" pad="2"></contactref><wire x1="6.27" y1="60.879999999999995" x2="10.08" y2="48.18" width="0" layer="19" extent="1-1"></wire><contactref element="U1" pad="GND.."></contactref><wire x1="10.08" y1="48.18" x2="45.64" y2="12.620000000000001" width="0" layer="19" extent="1-1"></wire><contactref element="BAT1" pad="-"></contactref><wire x1="45.64" y1="12.620000000000001" x2="5" y2="32.940000000000005" width="0" layer="19" extent="1-1"></wire></signal></signals>
 </board>
 </drawing>
